Commit message: feat: add prefix at links and joints

File: rbpodo_description/robots/rb_6dof.ros2_control.xacro (robot description, xacro)
@@ -15,21 +15,22 @@
         </xacro:unless>
       </hardware>
-      <xacro:macro name="configure_joint" params="joint_name torque_constant:=1">
+      <xacro:macro name="configure_joint" params="joint_name torque_constant:=1 initial_position:=0.0">
         <joint name="${joint_name}">
-          <param name="initial_position">0.0</param>
           <param name="torque_constant">${torque_constant}</param>
-          <command_interface name="effort"/>
+          <command_interface name="position"/>
           <command_interface name="velocity"/>
-          <command_interface name="position"/>
-          <state_interface name="position"/>
+          <state_interface name="position">
+            <param name="initial_value">${initial_position}</param>
+          </state_interface>
+          <state_interface name="velocity"/>
           <state_interface name="effort"/>
         </joint>
       </xacro:macro>
-      <xacro:configure_joint joint_name="${prefix}base" torque_constant="${torque_constants[0]}" />
-      <xacro:configure_joint joint_name="${prefix}shoulder" torque_constant="${torque_constants[1]}" />
-      <xacro:configure_joint joint_name="${prefix}elbow" torque_constant="${torque_constants[2]}" />
-      <xacro:configure_joint joint_name="${prefix}wrist1" torque_constant="${torque_constants[3]}" />
-      <xacro:configure_joint joint_name="${prefix}wrist2" torque_constant="${torque_constants[4]}" />
-      <xacro:configure_joint joint_name="${prefix}wrist3" torque_constant="${torque_constants[5]}" />
+      <xacro:configure_joint joint_name="${prefix}base"    torque_constant="${torque_constants[0]}" initial_position="2.212205"/>
+      <xacro:configure_joint joint_name="${prefix}shoulder" torque_constant="${torque_constants[1]}" initial_position="-0.258832"/>
+      <xacro:configure_joint joint_name="${prefix}elbow"    torque_constant="${torque_constants[2]}" initial_position="-1.894904"/>
+      <xacro:configure_joint joint_name="${prefix}wrist1"   torque_constant="${torque_constants[3]}" initial_position="-0.986460"/>
+      <xacro:configure_joint joint_name="${prefix}wrist2"   torque_constant="${torque_constants[4]}" initial_position="2.210809"/>
+      <xacro:configure_joint joint_name="${prefix}wrist3"   torque_constant="${torque_constants[5]}" initial_position="0.000175"/>
     </ros2_control>
   </xacro:macro>
